Commit message: Few Inertia Changes

File: src/my_robot_description/urdf/common_properties.xacro (robot description, xacro)
@@ -10,3 +10,11 @@
         <color rgba="0.7 0 0 1" />
     </material>
+    <xacro:macro name="box_inertia" params="m x y z o_rpy o_xyz">
+        <inertial>
+            <mass value="${m}"/>
+            <origin xyz="${o_xyz}" rpy="${o_rpy}"/>
+            <inertia ixx="${(m/12)*(y*y + z*z)}" ixy="0" ixz="0"
+                     iyy="${(m/12)*(x*x + z*z)}" iyz="0" izz="${(m/12)*(y*y + x*x)}" />
+        </inertial>
+    </xacro:macro>
 </robot>

File: src/my_robot_description/urdf/mobile_base.xacro (robot description, xacro)
@@ -1,7 +1,7 @@
 <?xml version="1.0"?>
 <robot xmlns:xacro="https://www.ros.org/wiki/xacro">
-    <xacro:property name="base_length" value="0.6" />
-    <xacro:property name="base_width" value="0.4" />
-    <xacro:property name="base_height" value="0.2" />
+    <xacro:property name="base_length" value="0.6" /> <!-- x-->
+    <xacro:property name="base_width" value="0.4" />  <!-- y-->
+    <xacro:property name="base_height" value="0.2" /> <!-- z-->
     <xacro:property name="wheel_radius" value="0.1" />
     <xacro:property name="wheel_length" value="0.05" />

Commit message: Added Sphere Inertia and Properites

File: src/my_robot_description/urdf/common_properties.xacro (robot description, xacro)
@@ -7,5 +7,5 @@
         <color rgba="0 0.7 0 1" />
     </material>
-     <material name="red">
+    <material name="red">
         <color rgba="0.7 0 0 1" />
     </material>
@@ -14,6 +14,12 @@
             <mass value="${m}"/>
             <origin xyz="${o_xyz}" rpy="${o_rpy}"/>
-            <inertia ixx="${(m/12)*(y*y + z*z)}" ixy="0" ixz="0"
-                     iyy="${(m/12)*(x*x + z*z)}" iyz="0" izz="${(m/12)*(y*y + x*x)}" />
+            <inertia ixx="${(m/12)*(y*y + z*z)}" ixy="0" ixz="0" iyy="${(m/12)*(x*x + z*z)}" iyz="0" izz="${(m/12)*(y*y + x*x)}" />
+        </inertial>
+    </xacro:macro>
+    <xacro:macro name="sphere_interia" params="m o_xyz o_rpy r">
+        <inertial>
+            <mass value="${m}" />
+            <origin xyz="${o_xyz}" rpy="${o_rpy}" />
+            <inertia ixx="${(2*m/5)*(r*r)}" ixy="0" ixz="0" iyy="${(2*m/5)*(r*r)}" iyz="0" izz="${(2*m/5)*(r*r)}" />
         </inertial>
     </xacro:macro>

File: src/my_robot_description/urdf/mobile_base.xacro (robot description, xacro)
@@ -1,10 +1,13 @@
 <?xml version="1.0"?>
 <robot xmlns:xacro="https://www.ros.org/wiki/xacro">
-    <xacro:property name="base_length" value="0.6" /> <!-- x-->
-    <xacro:property name="base_width" value="0.4" />  <!-- y-->
-    <xacro:property name="base_height" value="0.2" /> <!-- z-->
+    <xacro:property name="base_length" value="0.6" />
+    <!-- x-->
+    <xacro:property name="base_width" value="0.4" />
+    <!-- y-->
+    <xacro:property name="base_height" value="0.2" />
+    <!--z-->
     <xacro:property name="wheel_radius" value="0.1" />
     <xacro:property name="wheel_length" value="0.05" />
-   <xacro:macro name="wheel_link" params="prefix">
+    <xacro:macro name="wheel_link" params="prefix">
         <link name ="${prefix}_wheel_link">
             <visual>
@@ -20,5 +23,5 @@
         <visual>
             <geometry>
-            <!-- Metric system is used in urdf ros -->
+                <!-- Metric system is used in urdf ros -->
                 <box size="${base_length} ${base_width} ${base_height}"/>
                 <!--  length , width , height in meters-->
@@ -28,4 +31,5 @@
             <material name = "blue" />
         </visual>
+        <xacro:box_inertia m="5.0" o_xyz="0 0 0.1" o_rpy="0 0 0" x="${base_length}" y="${base_width}" z="${base_height}"/>
     </link>
     <link name="footprint">
@@ -37,8 +41,9 @@
             <origin xyz="0 0 0" rpy="0 0 0" />
             <geometry>
-               <sphere radius="0.05" />
+                <sphere radius="0.05" />
             </geometry>
             <material name="green" />
         </visual>
+        <xacro:sphere_interia m="1.0" o_xyz="0 0 0" o_rpy="0 0 0" r="0.05"/>
     </link>
     <joint name="base_joint" type="fixed">

Commit message: Made a Gazebo Launch File

File: src/my_robot_description/urdf/common_properties.xacro (robot description, xacro)
@@ -17,5 +17,5 @@
         </inertial>
     </xacro:macro>
-    <xacro:macro name="sphere_interia" params="m o_xyz o_rpy r">
+    <xacro:macro name="sphere_inertia" params="m o_xyz o_rpy r">
         <inertial>
             <mass value="${m}" />
@@ -24,3 +24,11 @@
         </inertial>
     </xacro:macro>
+    <xacro:macro name="wheel_inertia" params="m o_xyz o_rpy r h">
+        <inertial>
+            <mass value="${m}" />
+            <origin xyz="${o_xyz}" rpy="${o_rpy}" />
+            <inertia ixx="${(m/12)*(3*r*r + h*h)}" ixy="0" ixz="0" iyy="${(m/12)*(3*r*r + h*h)}" iyz="0"
+                     izz="${(m/12)*(3*r*r + h*h)}" />
+        </inertial>
+    </xacro:macro>
 </robot>

File: src/my_robot_description/urdf/mobile_base.xacro (robot description, xacro)
@@ -18,4 +18,11 @@
                 <material name = "red" />
             </visual>
+            <collision>
+                <geometry>
+                    <sphere radius="${wheel_radius}" />
+                    <origin xyz="0 0 0" rpy="0 0 0" />
+                </geometry>
+            </collision>
+            <xacro:wheel_inertia m="2.0" o_xyz="0 0 0" o_rpy="1.5708 0 0" r="${wheel_radius}" h="${wheel_length}" />
         </link>
     </xacro:macro>
@@ -26,9 +33,14 @@
                 <box size="${base_length} ${base_width} ${base_height}"/>
                 <!--  length , width , height in meters-->
-            </geometry>
-            <!-- rpy is roll,pitch,yaw -->
+            </geometry>            <!-- rpy is roll,pitch,yaw -->
             <origin xyz="0 0 0.1" rpy="0 0 0" />
             <material name = "blue" />
         </visual>
+        <collision>
+            <geometry>
+                <box size="${base_length} ${base_width} ${base_height}"/>
+            </geometry>
+            <origin xyz="0 0 0.1" rpy="0 0 0" />
+        </collision>
         <xacro:box_inertia m="5.0" o_xyz="0 0 0.1" o_rpy="0 0 0" x="${base_length}" y="${base_width}" z="${base_height}"/>
     </link>
@@ -45,5 +57,11 @@
             <material name="green" />
         </visual>
-        <xacro:sphere_interia m="1.0" o_xyz="0 0 0" o_rpy="0 0 0" r="0.05"/>
+        <collision>
+            <geometry>
+                <sphere radius="0.05" />
+                <origin xyz="0 0 0" rpy="0 0 0" />
+            </geometry>
+        </collision>
+        <xacro:sphere_inertia m="1.0" o_xyz="0 0 0" o_rpy="0 0 0" r="0.05"/>
     </link>
     <joint name="base_joint" type="fixed">
