Commit message: Inertia given and Camera module Added

File: src/my_robot_description/urdf/camera.xacro (robot description, xacro)
@@ -1,26 +1,28 @@
 <?xml version="1.0"?>
 <robot xmlns:xacro="https://www.ros.org/wiki/xacro">
-    <xacro:property name="camera_length" value="0.1" />
-    <xacro:property name="camera_height" value="0.1" />
-    <xacro:property name="camera_depth" value="0.5" />
+    <xacro:property name="camera_length" value="0.01" />
+    <xacro:property name="camera_width" value="0.1" />
+    <xacro:property name="camera_depth" value="0.05" />
     <link name="camera_link">
         <visual>
-            <origin xyz="0 0 0" rpy="0 0 0">
+            <origin xyz="0 0 0" rpy="0 0 0" />
                 <geometry>
-                    <box size="${camera_length} ${camera_height} ${camera_depth}" />
+                    <box size="${camera_length} ${camera_width} ${camera_depth}" />
                     <material name="red"/>
                 </geometry>
-            </visual>
-            <collision>
+        </visual>
+        <collision>
                 <geometry>
                     <box size="${camera_length} ${camera_height} ${camera_depth}"/>
                 </geometry>
                 <origin xyz="0 0 0" rpy="0 0 0" />
-            </collision>
+        </collision>
+        <xacro:box_inertia m="0.1" x="${camera_length}" y="${camera_width}" z="${camera_depth}"
+            o_rpy="0 0 0" o_xyz="0 0 0">
     </link>
     <joint name="base_camera_link" type="fixed">
         <parent link="base_link" />
         <child link="camera_link" />
-        <origin xyz="0 0 0" rpy="0 0 0">
+        <origin xyz="${base_length/2 + camera_length } 0 ${base_height/2}" rpy="0 0 0"/>
     </joint>
     </robot>

Commit message: Minor errors fixed file running

File: src/my_robot_description/urdf/camera.xacro (robot description, xacro)
@@ -14,15 +14,15 @@
         <collision>
                 <geometry>
-                    <box size="${camera_length} ${camera_height} ${camera_depth}"/>
+                    <box size="${camera_length} ${camera_width} ${camera_depth}"/>
                 </geometry>
                 <origin xyz="0 0 0" rpy="0 0 0" />
         </collision>
         <xacro:box_inertia m="0.1" x="${camera_length}" y="${camera_width}" z="${camera_depth}"
-            o_rpy="0 0 0" o_xyz="0 0 0">
+            o_rpy="0 0 0" o_xyz="0 0 0"/>
     </link>
     <joint name="base_camera_link" type="fixed">
         <parent link="base_link" />
         <child link="camera_link" />
-        <origin xyz="${base_length/2 + camera_length } 0 ${base_height/2}" rpy="0 0 0"/>
+        <origin xyz="${(base_length + camera_length )/2 } 0 ${base_height/2}" rpy="0 0 0"/>
     </joint>
     </robot>

Commit message: Gazebo Camera Plugin

File: src/my_robot_description/urdf/camera.xacro (robot description, xacro)
@@ -7,17 +7,16 @@
         <visual>
             <origin xyz="0 0 0" rpy="0 0 0" />
-                <geometry>
-                    <box size="${camera_length} ${camera_width} ${camera_depth}" />
-                    <material name="red"/>
-                </geometry>
+            <geometry>
+                <box size="${camera_length} ${camera_width} ${camera_depth}" />
+                <material name="red"/>
+            </geometry>
         </visual>
         <collision>
-                <geometry>
-                    <box size="${camera_length} ${camera_width} ${camera_depth}"/>
-                </geometry>
-                <origin xyz="0 0 0" rpy="0 0 0" />
+            <geometry>
+                <box size="${camera_length} ${camera_width} ${camera_depth}"/>
+            </geometry>
+            <origin xyz="0 0 0" rpy="0 0 0" />
         </collision>
-        <xacro:box_inertia m="0.1" x="${camera_length}" y="${camera_width}" z="${camera_depth}"
-            o_rpy="0 0 0" o_xyz="0 0 0"/>
+        <xacro:box_inertia m="0.1" x="${camera_length}" y="${camera_width}" z="${camera_depth}" o_rpy="0 0 0" o_xyz="0 0 0"/>
     </link>
     <joint name="base_camera_link" type="fixed">
@@ -26,3 +25,30 @@
         <origin xyz="${(base_length + camera_length )/2 } 0 ${base_height/2}" rpy="0 0 0"/>
     </joint>
+    <gazebo reference="camera_link">
+        <sensor name="camera" type="camera">
+            <camera>
+                <horizontal_fov>1.047</horizontal_fov>
+                <image>
+                    <width>640</width>
+                    <height>480</height>
+                    <format>R8G8B8</format>
+                </image>
+                <clip>
+                    <near>0.1</near>
+                    <far>15</far>
+                </clip>
+                <noise>
+                    <type>gaussian</type>
+                    <mean>0.0</mean>
+                    <stddev>0.007</stddev>
+                </noise>
+                <optical_frame_id>camera_link</optical_frame_id>
+                <camera_info_topic>camera/camera_info</camera_info_topic>
+            </camera>
+            <always_on>1</always_on>
+            <update_rate>30</update_rate>
+            <visualize>true</visualize>
+            <topic>camera/image_raw</topic>
+        </sensor>
+        </gazebo>
     </robot>

Commit message: Camera Optics Axis Changes

File: src/my_robot_description/urdf/camera.xacro (robot description, xacro)
@@ -25,4 +25,13 @@
         <origin xyz="${(base_length + camera_length )/2 } 0 ${base_height/2}" rpy="0 0 0"/>
     </joint>
+    <joint name="camera_optical_joint" type="fixed">
+    <!-- This joint was added with the knowledge of robo stac exchannge
+         to change the axis of camera optic so the blue line is removed feom the camera vision -->
+        <origin xyz="0 0 0" rpy="${-pi/2} 0 ${-pi/2}"/>
+        <parent link="camera_link"/>
+        <child link="camera_link_optical"/>
+    </joint>
+    <link name="camera_link_optical">
+    </link>
     <gazebo reference="camera_link">
         <sensor name="camera" type="camera">
@@ -43,5 +52,5 @@
                     <stddev>0.007</stddev>
                 </noise>
-                <optical_frame_id>camera_link</optical_frame_id>
+                <optical_frame_id>camera_link_optical</optical_frame_id>
                 <camera_info_topic>camera/camera_info</camera_info_topic>
             </camera>
@@ -51,4 +60,4 @@
             <topic>camera/image_raw</topic>
         </sensor>
-        </gazebo>
-    </robot>
+    </gazebo>
+</robot>
