Commit message: Rviz Setup done for testing

File: src/my_robot_description/urdf/arm_properties.xacro (robot description, xacro)
@@ -8,5 +8,5 @@
     </material>
     <material name="grey">
-        <color rgba="0.5 0.5 0.5 1" />
+        <color rgba="1 0.65 0 1" />
     </material>
     <xacro:property name="box_length" value="0.1" /> <!--x-->

File: src/my_robot_description/urdf/arm_visuals.xacro (robot description, xacro)
@@ -1,5 +1,5 @@
 <?xml version="1.0"?>
 <robot xmlns:xacro="https://www.ros.org/wiki/xacro">
-        <link name="arm_base_link">
+        <link name="base_link">
             <visual>
                 <origin xyz="0 0 0" rpy="0 0 0"/>
@@ -46,8 +46,8 @@
             </collision>
         </link>
-        <joint name="base_forearm_joint" type="revolute">
-            <parent link="arm_base_link" />
+        <joint name="base_link" type="revolute">
+            <parent link="base_link" />
             <child link="forearm_link" />
-            <origin xyz="0 0 0" rpy="0 0 0" />
+            <origin xyz="0 0 ${}" rpy="0 0 0" />
             <axis xyz="1 0 0" />
             <limit lower="0" upper="${pi/2}" effort="100" velocity="100" />
@@ -56,5 +56,5 @@
             <parent link="forearm_link" />
             <child link="hand_link" />
-            <origin xyz="0 0 0" rpy="0 0 0" />
+            <origin xyz="0 0 ${arm_length}" rpy="0 0 0" />
             <axis xyz="1 0 0" />
             <limit lower="0" upper="${pi/2}" effort="100" velocity="100" />

Commit message: Joints and URDF Design Done (Inertial LEft)

File: src/my_robot_description/urdf/arm_properties.xacro (robot description, xacro)
@@ -10,7 +10,8 @@
         <color rgba="1 0.65 0 1" />
     </material>
+<!-- left at setting up the joints origin -->
     <xacro:property name="box_length" value="0.1" /> <!--x-->
     <xacro:property name="box_width" value="0.1" />  <!--y-->
-    <xacro:property name="box_height" value="0.2" /> <!--z-->
+    <xacro:property name="box_height" value="0.02" /> <!--z-->
     <xacro:property name="box_mass" value="0.5" />   <!--box mass-->
     <xacro:property name="arm_width" value="0.02" />  <!--r-->

File: src/my_robot_description/urdf/arm_visuals.xacro (robot description, xacro)
@@ -3,5 +3,5 @@
         <link name="base_link">
             <visual>
-                <origin xyz="0 0 0" rpy="0 0 0"/>
+                <origin xyz="0 0 ${box_height/2}" rpy="0 0 0"/>
                 <geometry>
                     <box size="${box_length} ${box_width} ${box_height}" />
@@ -10,5 +10,5 @@
             </visual>
             <collision>
-                <origin xyz="0 0 0" rpy="0 0 0"/>
+                <origin xyz="0 0 ${box_height/2}" rpy="0 0 0"/>
                 <geometry>
                     <box size="${box_length} ${box_width} ${box_height}" />
@@ -18,5 +18,5 @@
         <link name="forearm_link">
             <visual>
-                <origin xyz="0 0 0" rpy="0 0 0" />
+                <origin xyz="0 0 ${arm_length/2}" rpy="0 0 0" />
                 <geometry>
                     <cylinder radius="${arm_width}" length="${arm_length}" />
@@ -25,5 +25,5 @@
             </visual>
             <collision>
-                <origin xyz="0 0 0" rpy="0 0 0" />
+                <origin xyz="0 0 ${arm_length/2}" rpy="0 0 0" />
                 <geometry>
                     <cylinder radius="${arm_width}" length="${arm_length}" />
@@ -33,5 +33,5 @@
         <link name="hand_link">
             <visual>
-                <origin xyz="0 0 0" rpy="0 0 0" />
+                <origin xyz="0 0 ${arm_length/2}" rpy="0 0 0" />
                 <geometry>
                     <cylinder radius="${arm_width}" length="${arm_length}" />
@@ -40,5 +40,5 @@
             </visual>
             <collision>
-                <origin xyz="0 0 0" rpy="0 0 0" />
+                <origin xyz="0 0 ${arm_length/2}" rpy="0 0 0" />
                 <geometry>
                     <cylinder radius="${arm_width}" length="${arm_length}" />
@@ -46,8 +46,8 @@
             </collision>
         </link>
-        <joint name="base_link" type="revolute">
+        <joint name="arm_base_link" type="revolute">
             <parent link="base_link" />
             <child link="forearm_link" />
-            <origin xyz="0 0 ${}" rpy="0 0 0" />
+            <origin xyz="0 0 ${box_height}" rpy="0 0 0" />
             <axis xyz="1 0 0" />
             <limit lower="0" upper="${pi/2}" effort="100" velocity="100" />

Commit message: Inertia to the Test arm

File: src/my_robot_description/urdf/arm_properties.xacro (robot description, xacro)
@@ -9,12 +9,36 @@
     <material name="grey">
         <color rgba="1 0.65 0 1" />
-    </material>
-<!-- left at setting up the joints origin -->
-    <xacro:property name="box_length" value="0.1" /> <!--x-->
-    <xacro:property name="box_width" value="0.1" />  <!--y-->
-    <xacro:property name="box_height" value="0.02" /> <!--z-->
-    <xacro:property name="box_mass" value="0.5" />   <!--box mass-->
-    <xacro:property name="arm_width" value="0.02" />  <!--r-->
-    <xacro:property name="arm_length" value="0.3" /> <!--h-->
-    <xacro:property name="arm_mass" value="0.3" />   <!--cylinder mass-->
+    </material>    <!-- left at setting up the joints origin -->
+    <xacro:property name="box_length" value="0.1" />
+    <!--x-->
+    <xacro:property name="box_width" value="0.1" />
+    <!--y-->
+    <xacro:property name="box_height" value="0.02"/>
+    <!--z-->
+    <xacro:property name="box_mass" value="0.5" />
+    <!--box mass-->
+    <xacro:property name="arm_width" value="0.02" />
+    <!--r-->
+    <xacro:property name="arm_length" value="0.3" />
+    <!--h-->
+    <xacro:property name="arm_mass" value="0.3" />
+    <!--cylinder mass-->
+    <xacro:macro name="arm_interia" params="o_xyz o_rpy">
+        <inertial>
+            <mass value="${arm_mass}" />
+            <origin xyz="${o_xyz}" rpy="${o_rpy}" />
+            <inertia ixx="${(1.0/12.0)*arm_mass*(3*arm_width*arm_width + arm_length*arm_length)}"
+                     iyy="${(1.0/12.0)*arm_mass*(3*arm_width*arm_width + arm_length*arm_length)}"
+                     izz="${(1.0/2.0)*arm_mass*arm_width*arm_width}" ixy="0" ixz="0" iyz="0"/>
+        </inertial>
+    </xacro:macro>
+    <xacro:macro name="arm_base_interia" params="o_xyz o_rpy ">
+        <inertial>
+            <mass value="${box_mass}" />
+            <origin xyz="${o_xyz}" rpy="${o_rpy}" />
+            <inertia ixx="${(box_mass/12)*(box_width*box_width+box_height*box_height)}"
+                     ixy="0" ixz="0" iyy="${(box_mass/12)*(box_length*box_length+box_height*box_height)}"
+                     iyz="0" izz="${(box_mass/12)*(box_length*box_length+box_width*box_width)}" />
+        </inertial>
+    </xacro:macro>
 </robot>

File: src/my_robot_description/urdf/arm_visuals.xacro (robot description, xacro)
@@ -15,4 +15,5 @@
                 </geometry>
             </collision>
+            <xacro:arm_base_interia o_rpy="0 0 ${box_height/2}" o_xyz="0 0 0" />
         </link>
         <link name="forearm_link">
@@ -30,4 +31,5 @@
                 </geometry>
             </collision>
+            <xacro:arm_interia o_rpy="0 0 0" o_xyz="0 0 ${arm_length/2}" />
         </link>
         <link name="hand_link">
@@ -45,4 +47,5 @@
                 </geometry>
             </collision>
+            <xacro:arm_interia o_rpy="0 0 0" o_xyz="0 0 ${arm_length/2}" />
         </link>
         <joint name="arm_base_link" type="revolute">
