Commit message: Making Gazebo

File: src/my_robot_description/urdf/arm_visuals.xacro (robot description, xacro)
@@ -1,5 +1,5 @@
 <?xml version="1.0"?>
 <robot xmlns:xacro="https://www.ros.org/wiki/xacro">
-        <link name="base_link">
+        <link name="base_arm_link">
             <visual>
                 <origin xyz="0 0 ${box_height/2}" rpy="0 0 0"/>
@@ -50,9 +50,10 @@
         </link>
         <joint name="arm_base_link" type="revolute">
-            <parent link="base_link" />
+            <parent link="base_arm_link" />
             <child link="forearm_link" />
             <origin xyz="0 0 ${box_height}" rpy="0 0 0" />
             <axis xyz="1 0 0" />
             <limit lower="0" upper="${pi/2}" effort="100" velocity="100" />
+            <dynamics friction="0.3" damping="0.3" />
         </joint>
         <joint name="forearm_arm_joint" type="revolute">
@@ -62,4 +63,5 @@
             <axis xyz="1 0 0" />
             <limit lower="0" upper="${pi/2}" effort="100" velocity="100" />
+            <dynamics friction="0.3" damping="0.3" />
         </joint>
     </robot>

File: src/my_robot_description/urdf/mobile_base.xacro (robot description, xacro)
@@ -85,3 +85,10 @@
         <axis xyz="0 1 0"/>
     </joint>
+    <joint name="base_left_wheel" type="">
+        <parent link="base_link" />
+        <child link="left_wheel_link" />
+        <origin xyz="${-base_length / 4.0} ${base_width / 2.0 + wheel_length/2} 0" rpy="0 0 0" />
+        <!-- 0.15 is the length 0.225 is height 0 is XYZ respective to height of base -->
+        <axis xyz="0 1 0"/>
+    </joint>
 </robot>

File: src/my_robot_description/urdf/my_robot.urdf.xacro (robot description, xacro)
@@ -4,4 +4,5 @@
     <xacro:include filename="mobile_base.xacro" />
     <xacro:include filename="mobile_base_gazeebo.xacro" />
+    <xacro:include filename="arm.xacro" />
     <xacro:include filename="camera.xacro" />
     <!-- the rpy works in radiance basically everything which works in degrees works in radiance -->
