Commit message: Gz arm bridge added  Publisher Working

File: src/my_robot_description/urdf/arm.xacro (robot description, xacro)
@@ -3,3 +3,4 @@
     <xacro:include filename="arm_properties.xacro" />
     <xacro:include filename="arm_visuals.xacro" />
+    <xacro:include filename="arm_gazebo.xacro" />
 </robot>

File: src/my_robot_description/urdf/arm_gazebo.xacro (robot description, xacro)
@@ -1,3 +1,20 @@
 <?xml version="1.0"?>
-<robot name="mesh_robot" xmlns:xacro="https://www.ros.org/wiki/xacro">
+<robot xmlns:xacro="https://www.ros.org/wiki/xacro">
+    <gazebo>
+        <plugin filename="gz-sim-joint-position-controller-system" name="gz::sim::systems::JointPositionController">
+            <joint_name>arm_base_link</joint_name>
+        </plugin>
+    </gazebo>
+    <gazebo>
+        <plugin filename="gz-sim-joint-position-controller-system" name="gz::sim::systems::JointPositionController">
+            <joint_name>forearm_arm_joint</joint_name>
+        </plugin>
+    </gazebo>
+    <gazebo>
+        <plugin filename="gz-sim-joint-state-publisher-system"
+                name="gz::sim::systems::JointStatePublisher">
+                <joint_name>arm_base_link</joint_name>
+                <joint_name>forearm_arm_joint</joint_name>
+        </plugin>
+    </gazebo>
 </robot>

File: src/my_robot_description/urdf/arm_properties.xacro (robot description, xacro)
@@ -16,5 +16,5 @@
     <xacro:property name="box_height" value="0.02"/>
     <!--z-->
-    <xacro:property name="box_mass" value="0.5" />
+    <xacro:property name="box_mass" value="5.0" />
     <!--box mass-->
     <xacro:property name="arm_width" value="0.02" />
