Commit message: Setting up Gazeebo Plugings

File: src/my_robot_description/urdf/mobile_base.xacro (robot description, xacro)
@@ -1,13 +1,11 @@
 <?xml version="1.0"?>
 <robot xmlns:xacro="https://www.ros.org/wiki/xacro">
-    <xacro:property name="base_length" value="0.6" />
-    <!-- x-->
-    <xacro:property name="base_width" value="0.4" />
-    <!-- y-->
-    <xacro:property name="base_height" value="0.2" />
-    <!--z-->
+    <xacro:property name="base_length" value="0.6" /><!-- x-->
+    <xacro:property name="base_width" value="0.4" /><!-- y-->
+    <xacro:property name="base_height" value="0.2" /><!--z-->
     <xacro:property name="wheel_radius" value="0.1" />
     <xacro:property name="wheel_length" value="0.05" />
     <xacro:macro name="wheel_link" params="prefix">
+        <link name="footprint"/>
         <link name ="${prefix}_wheel_link">
             <visual>
@@ -44,6 +42,4 @@
         </collision>
         <xacro:box_inertia m="5.0" o_xyz="0 0 0.1" o_rpy="0 0 0" x="${base_length}" y="${base_width}" z="${base_height}"/>
-    </link>
-    <link name="footprint">
     </link>
     <xacro:wheel_link prefix="right"/>

File: src/my_robot_description/urdf/my_robot.urdf.xacro (robot description, xacro)
@@ -3,4 +3,5 @@
     <xacro:include filename="common_properties.xacro" />
     <xacro:include filename="mobile_base.xacro" />
+    <xacro:include filename="mobile_base_gazeebo.xacro" />
     <!-- the rpy works in radiance basically everything which works in degrees works in radiance -->
     <!-- Every Measurement is done in Meters and not CMs MM or Kms -->

Commit message: some how the Plugins FIxed by single line change

File: src/my_robot_description/urdf/mobile_base.xacro (robot description, xacro)
@@ -7,5 +7,4 @@
     <xacro:property name="wheel_length" value="0.05" />
     <xacro:macro name="wheel_link" params="prefix">
-        <link name="footprint"/>
         <link name ="${prefix}_wheel_link">
             <visual>
@@ -42,4 +41,6 @@
         </collision>
         <xacro:box_inertia m="5.0" o_xyz="0 0 0.1" o_rpy="0 0 0" x="${base_length}" y="${base_width}" z="${base_height}"/>
+    </link>
+    <link name="footprint">
     </link>
     <xacro:wheel_link prefix="right"/>

File: src/my_robot_description/urdf/mobile_base_gazeebo.xacro (robot description, xacro)
@@ -1,5 +1,4 @@
 <?xml version="1.0"?>
-<robot name="mesh_robot"
-    xmlns:xacro="https://www.ros.org/wiki/xacro">
+<robot name="mesh_robot" xmlns:xacro="https://www.ros.org/wiki/xacro">
             <!-- Name comes from same github repo
                         at the end of file type cc the name is avaliable -->
@@ -24,5 +23,4 @@
         <plugin filename="gz-sim-joint-state-publisher-system"
                 name="gz::sim::systems::JointStatePublisher">
-                <topic>My_robot10<topic>
                 <joint_name>base_left_wheel</joint_name>
                 <joint_name>base_right_wheel</joint_name>

Commit message: F_OLD_DATA ignoring data from the past for frame base_footprint at time 3473.659000 according to authority Authority undetectable Issue Caused

File: src/my_robot_description/urdf/mobile_base.xacro (robot description, xacro)
@@ -42,6 +42,5 @@
         <xacro:box_inertia m="5.0" o_xyz="0 0 0.1" o_rpy="0 0 0" x="${base_length}" y="${base_width}" z="${base_height}"/>
     </link>
-    <link name="footprint">
-    </link>
+    <link name="base_footprint" ></link>
     <xacro:wheel_link prefix="right"/>
     <xacro:wheel_link prefix="left"/>
@@ -63,9 +62,9 @@
     </link>
     <joint name="base_joint" type="fixed">
-        <parent link="footprint" />
+        <parent link="base_footprint" />
         <child link="base_link" />
         <origin xyz="0 0 ${wheel_radius}" rpy="0 0 0" />
     </joint>
-    <joint name="base_sphere_joint" type="continuous">
+    <joint name="base_sphere_joint" type="fixed">
         <parent link="base_link" />
         <child link="sphere_link" />

File: src/my_robot_description/urdf/mobile_base_gazeebo.xacro (robot description, xacro)
@@ -1,9 +1,4 @@
 <?xml version="1.0"?>
 <robot name="mesh_robot" xmlns:xacro="https://www.ros.org/wiki/xacro">
-            <!-- Name comes from same github repo
-                        at the end of file type cc the name is avaliable -->
-            <!-- The name gz-sim-diff-drive-system came from the gz-sim github repo
-                gz-sim is compulsory system is compulsoly just we need to
-                put the name like this  -->
     <gazebo reference="sphere_link">
         <mu1 value="0.1"/>
@@ -17,5 +12,5 @@
                 <wheel_radius>0.1</wheel_radius>
                 <frame_id>odom</frame_id>
-                <child_frame_id>footprint</child_frame_id>
+                <child_frame_id>base_footprint</child_frame_id>
         </plugin>
     </gazebo>

Commit message: Robo arm and Vehical Connected and works

File: src/my_robot_description/urdf/mobile_base.xacro (robot description, xacro)
@@ -85,10 +85,3 @@
         <axis xyz="0 1 0"/>
     </joint>
-    <joint name="base_left_wheel" type="">
-        <parent link="base_link" />
-        <child link="left_wheel_link" />
-        <origin xyz="${-base_length / 4.0} ${base_width / 2.0 + wheel_length/2} 0" rpy="0 0 0" />
-        <!-- 0.15 is the length 0.225 is height 0 is XYZ respective to height of base -->
-        <axis xyz="0 1 0"/>
-    </joint>
 </robot>

File: src/my_robot_description/urdf/my_robot.urdf.xacro (robot description, xacro)
@@ -8,3 +8,9 @@
     <!-- the rpy works in radiance basically everything which works in degrees works in radiance -->
     <!-- Every Measurement is done in Meters and not CMs MM or Kms -->
+    <joint name="mesh_robot_arm_link" type="fixed">
+        <parent link="base_link" />
+        <child link="base_arm_link" />
+        <origin xyz="0 0 ${base_height}" rpy="0 0 1.5708" />
+        <axis xyz="0 0 0"/>
+    </joint>
    </robot>
