Commit message: Adding Diff Drive and Controller

File: src/my_robot_description/urdf/my_robot.urdf.xacro (robot description, xacro)
@@ -4,9 +4,9 @@
     <xacro:include filename="mobile_base.xacro" />
     <xacro:include filename="mobile_base_gazeebo.xacro" />
-    <xacro:include filename="arm.xacro" />
+    <!-- <xacro:include filename="arm.xacro" /> when i will need the arm i will enable this -->
     <xacro:include filename="camera.xacro" />
     <!-- the rpy works in radiance basically everything which works in degrees works in radiance -->
     <!-- Every Measurement is done in Meters and not CMs MM or Kms -->
-    <joint name="mesh_robot_arm_link" type="fixed">
+    <!-- <joint name="mesh_robot_arm_link" type="fixed">
         <parent link="base_link" />
         <child link="base_arm_link" />
@@ -14,3 +14,4 @@
         <axis xyz="0 0 0"/>
     </joint>
+    this joint is also related to the arm of the robot-->
    </robot>
